File: PCBs/PCH-1XXX/PCH-1000JIG_THT/Kicad/PCH-1xxxJIG_THT_1.4.kicad_pcb (KiCad board)
At the start: 2 copper layers, 73.7 x 61 mm, 15 parts, among them U1 Vita_Connector

Commit message: changed UDC silkscreen label
Parts:
- renumbered U1 to UDC
Changed lines of the file:
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@@
     (at 87.36 84.26)
     (attr smd)
-    (fp_text reference "U1" (at 5.064 -1.924) (layer "F.SilkS")
+    (fp_text reference "UDC" (at 3.14 -1.924) (layer "F.SilkS")
         (effects (font (size 1.143 1.143) (thickness 0.152)) (justify left))
     )
