File: PCBs/PCH-2XXX/PCH-2xxxJIG_0805_Nano_5V/Kicad/PCH-2xxxJIG_0805_Nano.kicad_pcb (KiCad board)
At the start: 2 copper layers, 20.1 x 14 mm, 13 parts

Commit message: Fixed a bad bridge
Routing:
- net (no net): track 114.7 -> 112.2 mm
Other:
- board text added: "PCH-2XXXJIG Rev 1.2 by Mathieulh"
- board text removed: "PCH-2XXXJIG Rev 1.1 by Mathieulh"
Changed lines of the file:
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@@
   (gr_rect (start 58.86 31) (end 79 45.04)
     (stroke (width 0.1) (type default)) (fill none) (layer "Edge.Cuts"))
-  (gr_text "PCH-2XXXJIG Rev 1.1 by Mathieulh" (at 63.5 40.64) (layer "B.SilkS")
+  (gr_text "PCH-2XXXJIG Rev 1.2 by Mathieulh" (at 63.5 40.64) (layer "B.SilkS")
     (effects (font (size 0.7 0.5) (thickness 0.1) bold) (justify left bottom))
   )
@@
   )
   (segment (start 78 38.1) (end 76.2 38.1) (width 0.2) (layer "F.Cu") (net 0))
-  (segment (start 76.2 38.1) (end 76.2 40.64) (width 0.2) (layer "F.Cu") (net 0))
   (segment (start 72.12 39.4) (end 74.96 39.4) (width 0.2) (layer "F.Cu") (net 0))
   (segment (start 73.66 40.64) (end 76.2 40.64) (width 0.2) (layer "F.Cu") (net 0))
