File: PCBs/JIG SWITCH/Kicad/JIG SWITCH.kicad_pcb (KiCad board)
At the start: 2 copper layers, 99.1 x 88.9 mm, 22 parts, among them U3 12pad

Commit message: Fixed resistor value for 5V circuit
Other:
- board text added: "R1 = 7.5K R2 = 10K R3 = 0 R4 = 0 R5 = 0 R6 = 7.5K R7 = 2K R8 = 2K R9 = 1K"
- board text removed: "R1 = 7.5K R2 = 10K R3 = 0 R4 = 0 R5 = 0 R6 = 7.5K R7 = 2K R8 = 1K R9 = 1K"
Changed lines of the file:
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@@
     (effects (font (size 1.5 1.5) (thickness 0.3) bold) (justify left bottom))
   )
-  (gr_text "R1 = 7.5K\nR2 = 10K\nR3 = 0\nR4 = 0\nR5 = 0\nR6 = 7.5K\nR7 = 2K\nR8 = 1K\nR9 = 1K" (at 33.02 115.57) (layer "F.SilkS")
+  (gr_text "R1 = 7.5K\nR2 = 10K\nR3 = 0\nR4 = 0\nR5 = 0\nR6 = 7.5K\nR7 = 2K\nR8 = 2K\nR9 = 1K" (at 33.02 115.57) (layer "F.SilkS")
     (effects (font (size 2 2) (thickness 0.1)) (justify left bottom))
   )

Commit message: Added a warning label at the back of the board
Other:
- board text added: "** CAUTION ** Some UART modules advertised as 5V or with a jumper to 5V do NOT shift the power levels for UART TX/RX which will operate at 3.3V, Please measure voltage using a multimeter on your UART module between TX and GND. if it runs at 3.3V Replace R1 to a 1K ohms resistor."
Changed lines of the file:
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@@
     )
   )
+  (gr_rect (start 33.02 35.56) (end 124.46 48.26)
+    (stroke (width 0.2) (type default)) (fill none) (layer "B.SilkS"))
   (gr_rect (start 33.02 82.55) (end 50.8 115.57)
     (stroke (width 0.2) (type default)) (fill none) (layer "F.SilkS"))
@@
   (gr_rect (start 31.06 29.9) (end 130.12 118.8)
     (stroke (width 0.1) (type default)) (fill none) (layer "Edge.Cuts"))
+  (gr_text "** CAUTION ** \n\n\nSome UART modules advertised as 5V or with a jumper to 5V do NOT shift the power levels for UART TX/RX \nwhich will operate at 3.3V, Please measure voltage using a multimeter on your UART module between TX and GND.\nif it runs at 3.3V Replace R1 to a 1K ohms resistor." (at 121.92 45.72) (layer "B.SilkS")
+    (effects (font (size 1 1) (thickness 0.2) bold) (justify left bottom mirror))
+  )
   (gr_text "PCH JIG MULTI SWITCH BOARD 2.0\nBy Mathieulh" (at 83.82 37.52) (layer "F.SilkS")
     (effects (font (size 1.5 1.5) (thickness 0.3) bold) (justify left bottom))
